File: hardware/sd-board/sd-board.kicad_sch (KiCad schematic)
At the start: 13 parts, among them J1 TF-01A push-push, J2 FFC 6P 0.5mm, U1 74LVC1G04

Commit message: feat(hardware): SD board v3 held by two of the FM-1's own screws (38.1 mm apart, measured; the case's poles 6.8 mm, measured), the inverter and its parts moved into the strip under the FFC socket so the foot is 22 mm wide, not 31 (the battery moves less); CS and 3V3 reach the card on the bottom round the lower screw; FFC order MOSI CLK MISO GND 3V3 CS; MEASUREMENTS.md (measured vs photo), a 3D-print mockup.stl and a 1:1 template; DRC 0, nets 0 differ
Parts:
- removed H4: M2, MountingHole:MountingHole_2.2mm_M2, symbol Mechanical:MountingHole
- H1, H2: footprint MountingHole:MountingHole_2.2mm_M2 -> MountingHole:MountingHole_2.7mm_M2.5
Connections:
- net 3V3: now also J2.5 (Pin_5); no longer J2.3 (Pin_3)
- net CLK: now also J2.2 (Pin_2); no longer J2.4 (Pin_4)
- net GND: now also J2.4 (Pin_4); no longer J2.5 (Pin_5)
- net LCD_CS: now also J2.6 (Pin_6); no longer J2.1 (Pin_1)
- net MISO: now also J2.3 (Pin_3); no longer J2.6 (Pin_6)
- net MOSI: now also J2.1 (Pin_1); no longer J2.2 (Pin_2)
Changed lines of the file:
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@@
 (label "3V3" (at 76.2 128.27 270) (effects (font (size 1.27 1.27)) (justify left bottom)))
 (symbol (lib_id "Connector_Generic_MountingPin:Conn_01x06_MountingPin") (at 231.14 88.9 0) (unit 1) (exclude_from_sim no) (in_bom yes) (on_board yes) (dnp no) (property "Reference" "J2" (at 231.14 74.9 0) (effects (font (size 1.27 1.27)))) (property "Value" "FFC 6P 0.5mm" (at 231.14 102.9 0) (effects (font (size 1.27 1.27)))) (property "Footprint" "sdboard:FPC-SMD_6P-P0.50_XUNPU_FPC-05F-6PH20" (at 231.14 88.9 0) (effects (font (size 1.27 1.27)) (hide yes))) (property "Datasheet" "" (at 231.14 88.9 0) (effects (font (size 1.27 1.27)) (hide yes))) (property "LCSC" "C2856796" (at 231.14 88.9 0) (effects (font (size 1.27 1.27)) (hide yes))) (pin "1") (pin "2") (pin "3") (pin "4") (pin "5") (pin "6") (pin "MP") (instances (project "sd-board" (path "/766c70bd-1acb-59f5-b703-96c0315a8041" (reference "J2") (unit 1)))))
-(label "LCD_CS" (at 226.06 83.82 180) (effects (font (size 1.27 1.27)) (justify right bottom)))
-(label "MOSI" (at 226.06 86.36 180) (effects (font (size 1.27 1.27)) (justify right bottom)))
-(label "3V3" (at 226.06 88.9 180) (effects (font (size 1.27 1.27)) (justify right bottom)))
-(label "CLK" (at 226.06 91.44 180) (effects (font (size 1.27 1.27)) (justify right bottom)))
-(label "GND" (at 226.06 93.98 180) (effects (font (size 1.27 1.27)) (justify right bottom)))
-(label "MISO" (at 226.06 96.52 180) (effects (font (size 1.27 1.27)) (justify right bottom)))
+(label "MOSI" (at 226.06 83.82 180) (effects (font (size 1.27 1.27)) (justify right bottom)))
+(label "CLK" (at 226.06 86.36 180) (effects (font (size 1.27 1.27)) (justify right bottom)))
+(label "MISO" (at 226.06 88.9 180) (effects (font (size 1.27 1.27)) (justify right bottom)))
+(label "GND" (at 226.06 91.44 180) (effects (font (size 1.27 1.27)) (justify right bottom)))
+(label "3V3" (at 226.06 93.98 180) (effects (font (size 1.27 1.27)) (justify right bottom)))
+(label "LCD_CS" (at 226.06 96.52 180) (effects (font (size 1.27 1.27)) (justify right bottom)))
 (label "GND" (at 231.14 101.6 270) (effects (font (size 1.27 1.27)) (justify left bottom)))
-(symbol (lib_id "Mechanical:MountingHole") (at 215.9 149.86 0) (unit 1) (exclude_from_sim no) (in_bom no) (on_board yes) (dnp no) (property "Reference" "H1" (at 215.9 135.86 0) (effects (font (size 1.27 1.27)))) (property "Value" "M2" (at 215.9 163.86 0) (effects (font (size 1.27 1.27)))) (property "Footprint" "MountingHole:MountingHole_2.2mm_M2" (at 215.9 149.86 0) (effects (font (size 1.27 1.27)) (hide yes))) (property "Datasheet" "" (at 215.9 149.86 0) (effects (font (size 1.27 1.27)) (hide yes))) (property "LCSC" "" (at 215.9 149.86 0) (effects (font (size 1.27 1.27)) (hide yes)))  (instances (project "sd-board" (path "/766c70bd-1acb-59f5-b703-96c0315a8041" (reference "H1") (unit 1)))))
-(symbol (lib_id "Mechanical:MountingHole") (at 231.14 149.86 0) (unit 1) (exclude_from_sim no) (in_bom no) (on_board yes) (dnp no) (property "Reference" "H2" (at 231.14 135.86 0) (effects (font (size 1.27 1.27)))) (property "Value" "M2" (at 231.14 163.86 0) (effects (font (size 1.27 1.27)))) (property "Footprint" "MountingHole:MountingHole_2.2mm_M2" (at 231.14 149.86 0) (effects (font (size 1.27 1.27)) (hide yes))) (property "Datasheet" "" (at 231.14 149.86 0) (effects (font (size 1.27 1.27)) (hide yes))) (property "LCSC" "" (at 231.14 149.86 0) (effects (font (size 1.27 1.27)) (hide yes)))  (instances (project "sd-board" (path "/766c70bd-1acb-59f5-b703-96c0315a8041" (reference "H2") (unit 1)))))
+(symbol (lib_id "Mechanical:MountingHole") (at 215.9 149.86 0) (unit 1) (exclude_from_sim no) (in_bom no) (on_board yes) (dnp no) (property "Reference" "H1" (at 215.9 135.86 0) (effects (font (size 1.27 1.27)))) (property "Value" "M2" (at 215.9 163.86 0) (effects (font (size 1.27 1.27)))) (property "Footprint" "MountingHole:MountingHole_2.7mm_M2.5" (at 215.9 149.86 0) (effects (font (size 1.27 1.27)) (hide yes))) (property "Datasheet" "" (at 215.9 149.86 0) (effects (font (size 1.27 1.27)) (hide yes))) (property "LCSC" "" (at 215.9 149.86 0) (effects (font (size 1.27 1.27)) (hide yes)))  (instances (project "sd-board" (path "/766c70bd-1acb-59f5-b703-96c0315a8041" (reference "H1") (unit 1)))))
+(symbol (lib_id "Mechanical:MountingHole") (at 231.14 149.86 0) (unit 1) (exclude_from_sim no) (in_bom no) (on_board yes) (dnp no) (property "Reference" "H2" (at 231.14 135.86 0) (effects (font (size 1.27 1.27)))) (property "Value" "M2" (at 231.14 163.86 0) (effects (font (size 1.27 1.27)))) (property "Footprint" "MountingHole:MountingHole_2.7mm_M2.5" (at 231.14 149.86 0) (effects (font (size 1.27 1.27)) (hide yes))) (property "Datasheet" "" (at 231.14 149.86 0) (effects (font (size 1.27 1.27)) (hide yes))) (property "LCSC" "" (at 231.14 149.86 0) (effects (font (size 1.27 1.27)) (hide yes)))  (instances (project "sd-board" (path "/766c70bd-1acb-59f5-b703-96c0315a8041" (reference "H2") (unit 1)))))
 (symbol (lib_id "Mechanical:MountingHole") (at 243.84 149.86 0) (unit 1) (exclude_from_sim no) (in_bom no) (on_board yes) (dnp no) (property "Reference" "H3" (at 243.84 135.86 0) (effects (font (size 1.27 1.27)))) (property "Value" "M2" (at 243.84 163.86 0) (effects (font (size 1.27 1.27)))) (property "Footprint" "MountingHole:MountingHole_2.2mm_M2" (at 243.84 149.86 0) (effects (font (size 1.27 1.27)) (hide yes))) (property "Datasheet" "" (at 243.84 149.86 0) (effects (font (size 1.27 1.27)) (hide yes))) (property "LCSC" "" (at 243.84 149.86 0) (effects (font (size 1.27 1.27)) (hide yes)))  (instances (project "sd-board" (path "/766c70bd-1acb-59f5-b703-96c0315a8041" (reference "H3") (unit 1)))))
-(symbol (lib_id "Mechanical:MountingHole") (at 259.08 149.86 0) (unit 1) (exclude_from_sim no) (in_bom no) (on_board yes) (dnp no) (property "Reference" "H4" (at 259.08 135.86 0) (effects (font (size 1.27 1.27)))) (property "Value" "M2" (at 259.08 163.86 0) (effects (font (size 1.27 1.27)))) (property "Footprint" "MountingHole:MountingHole_2.2mm_M2" (at 259.08 149.86 0) (effects (font (size 1.27 1.27)) (hide yes))) (property "Datasheet" "" (at 259.08 149.86 0) (effects (font (size 1.27 1.27)) (hide yes))) (property "LCSC" "" (at 259.08 149.86 0) (effects (font (size 1.27 1.27)) (hide yes)))  (instances (project "sd-board" (path "/766c70bd-1acb-59f5-b703-96c0315a8041" (reference "H4") (unit 1)))))
 (symbol (lib_id "power:PWR_FLAG") (at 40.64 149.86 0) (unit 1) (exclude_from_sim no) (in_bom no) (on_board no) (dnp no) (property "Reference" "#FLG01" (at 40.64 135.86 0) (effects (font (size 1.27 1.27)) (hide yes))) (property "Value" "PWR_FLAG" (at 40.64 163.86 0) (effects (font (size 1.27 1.27)) (hide yes))) (property "Footprint" "" (at 40.64 149.86 0) (effects (font (size 1.27 1.27)) (hide yes))) (property "Datasheet" "" (at 40.64 149.86 0) (effects (font (size 1.27 1.27)) (hide yes))) (property "LCSC" "" (at 40.64 149.86 0) (effects (font (size 1.27 1.27)) (hide yes))) (pin "1") (instances (project "sd-board" (path "/766c70bd-1acb-59f5-b703-96c0315a8041" (reference "#FLG01") (unit 1)))))
 (label "3V3" (at 40.64 149.86 0) (effects (font (size 1.27 1.27)) (justify left bottom)))

Commit message: feat(hardware): SD board v3: the tie hole dropped (the two FM-1 screws hold it), the foot trimmed to the card socket (22 x 22.6 mm past the lower screw; the user's cover sketch shows the same L)
Parts:
- removed H3: M2, MountingHole:MountingHole_2.2mm_M2, symbol Mechanical:MountingHole
- H1, H2: value M2 -> M2.5
Changed lines of the file:
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@@
 (label "LCD_CS" (at 226.06 96.52 180) (effects (font (size 1.27 1.27)) (justify right bottom)))
 (label "GND" (at 231.14 101.6 270) (effects (font (size 1.27 1.27)) (justify left bottom)))
-(symbol (lib_id "Mechanical:MountingHole") (at 215.9 149.86 0) (unit 1) (exclude_from_sim no) (in_bom no) (on_board yes) (dnp no) (property "Reference" "H1" (at 215.9 135.86 0) (effects (font (size 1.27 1.27)))) (property "Value" "M2" (at 215.9 163.86 0) (effects (font (size 1.27 1.27)))) (property "Footprint" "MountingHole:MountingHole_2.7mm_M2.5" (at 215.9 149.86 0) (effects (font (size 1.27 1.27)) (hide yes))) (property "Datasheet" "" (at 215.9 149.86 0) (effects (font (size 1.27 1.27)) (hide yes))) (property "LCSC" "" (at 215.9 149.86 0) (effects (font (size 1.27 1.27)) (hide yes)))  (instances (project "sd-board" (path "/766c70bd-1acb-59f5-b703-96c0315a8041" (reference "H1") (unit 1)))))
-(symbol (lib_id "Mechanical:MountingHole") (at 231.14 149.86 0) (unit 1) (exclude_from_sim no) (in_bom no) (on_board yes) (dnp no) (property "Reference" "H2" (at 231.14 135.86 0) (effects (font (size 1.27 1.27)))) (property "Value" "M2" (at 231.14 163.86 0) (effects (font (size 1.27 1.27)))) (property "Footprint" "MountingHole:MountingHole_2.7mm_M2.5" (at 231.14 149.86 0) (effects (font (size 1.27 1.27)) (hide yes))) (property "Datasheet" "" (at 231.14 149.86 0) (effects (font (size 1.27 1.27)) (hide yes))) (property "LCSC" "" (at 231.14 149.86 0) (effects (font (size 1.27 1.27)) (hide yes)))  (instances (project "sd-board" (path "/766c70bd-1acb-59f5-b703-96c0315a8041" (reference "H2") (unit 1)))))
-(symbol (lib_id "Mechanical:MountingHole") (at 243.84 149.86 0) (unit 1) (exclude_from_sim no) (in_bom no) (on_board yes) (dnp no) (property "Reference" "H3" (at 243.84 135.86 0) (effects (font (size 1.27 1.27)))) (property "Value" "M2" (at 243.84 163.86 0) (effects (font (size 1.27 1.27)))) (property "Footprint" "MountingHole:MountingHole_2.2mm_M2" (at 243.84 149.86 0) (effects (font (size 1.27 1.27)) (hide yes))) (property "Datasheet" "" (at 243.84 149.86 0) (effects (font (size 1.27 1.27)) (hide yes))) (property "LCSC" "" (at 243.84 149.86 0) (effects (font (size 1.27 1.27)) (hide yes)))  (instances (project "sd-board" (path "/766c70bd-1acb-59f5-b703-96c0315a8041" (reference "H3") (unit 1)))))
+(symbol (lib_id "Mechanical:MountingHole") (at 215.9 149.86 0) (unit 1) (exclude_from_sim no) (in_bom no) (on_board yes) (dnp no) (property "Reference" "H1" (at 215.9 135.86 0) (effects (font (size 1.27 1.27)))) (property "Value" "M2.5" (at 215.9 163.86 0) (effects (font (size 1.27 1.27)))) (property "Footprint" "MountingHole:MountingHole_2.7mm_M2.5" (at 215.9 149.86 0) (effects (font (size 1.27 1.27)) (hide yes))) (property "Datasheet" "" (at 215.9 149.86 0) (effects (font (size 1.27 1.27)) (hide yes))) (property "LCSC" "" (at 215.9 149.86 0) (effects (font (size 1.27 1.27)) (hide yes)))  (instances (project "sd-board" (path "/766c70bd-1acb-59f5-b703-96c0315a8041" (reference "H1") (unit 1)))))
+(symbol (lib_id "Mechanical:MountingHole") (at 231.14 149.86 0) (unit 1) (exclude_from_sim no) (in_bom no) (on_board yes) (dnp no) (property "Reference" "H2" (at 231.14 135.86 0) (effects (font (size 1.27 1.27)))) (property "Value" "M2.5" (at 231.14 163.86 0) (effects (font (size 1.27 1.27)))) (property "Footprint" "MountingHole:MountingHole_2.7mm_M2.5" (at 231.14 149.86 0) (effects (font (size 1.27 1.27)) (hide yes))) (property "Datasheet" "" (at 231.14 149.86 0) (effects (font (size 1.27 1.27)) (hide yes))) (property "LCSC" "" (at 231.14 149.86 0) (effects (font (size 1.27 1.27)) (hide yes)))  (instances (project "sd-board" (path "/766c70bd-1acb-59f5-b703-96c0315a8041" (reference "H2") (unit 1)))))
 (symbol (lib_id "power:PWR_FLAG") (at 40.64 149.86 0) (unit 1) (exclude_from_sim no) (in_bom no) (on_board no) (dnp no) (property "Reference" "#FLG01" (at 40.64 135.86 0) (effects (font (size 1.27 1.27)) (hide yes))) (property "Value" "PWR_FLAG" (at 40.64 163.86 0) (effects (font (size 1.27 1.27)) (hide yes))) (property "Footprint" "" (at 40.64 149.86 0) (effects (font (size 1.27 1.27)) (hide yes))) (property "Datasheet" "" (at 40.64 149.86 0) (effects (font (size 1.27 1.27)) (hide yes))) (property "LCSC" "" (at 40.64 149.86 0) (effects (font (size 1.27 1.27)) (hide yes))) (pin "1") (instances (project "sd-board" (path "/766c70bd-1acb-59f5-b703-96c0315a8041" (reference "#FLG01") (unit 1)))))
 (label "3V3" (at 40.64 149.86 0) (effects (font (size 1.27 1.27)) (justify left bottom)))

Commit message: feat(hardware): SD board v3: the back cover's poles pass through it (the user): two 5.5 mm holes (pole 5.2 from a photo + 0.3), centres 38.1 - 5.2 apart (38.1 over the outer edges, measured); the strip's top 1.5 mm above the upper hole
Parts:
- H1, H2: value M2.5 -> pole; footprint MountingHole:MountingHole_2.7mm_M2.5 -> sdboard:PoleHole
Changed lines of the file:
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@@
 (label "LCD_CS" (at 226.06 96.52 180) (effects (font (size 1.27 1.27)) (justify right bottom)))
 (label "GND" (at 231.14 101.6 270) (effects (font (size 1.27 1.27)) (justify left bottom)))
-(symbol (lib_id "Mechanical:MountingHole") (at 215.9 149.86 0) (unit 1) (exclude_from_sim no) (in_bom no) (on_board yes) (dnp no) (property "Reference" "H1" (at 215.9 135.86 0) (effects (font (size 1.27 1.27)))) (property "Value" "M2.5" (at 215.9 163.86 0) (effects (font (size 1.27 1.27)))) (property "Footprint" "MountingHole:MountingHole_2.7mm_M2.5" (at 215.9 149.86 0) (effects (font (size 1.27 1.27)) (hide yes))) (property "Datasheet" "" (at 215.9 149.86 0) (effects (font (size 1.27 1.27)) (hide yes))) (property "LCSC" "" (at 215.9 149.86 0) (effects (font (size 1.27 1.27)) (hide yes)))  (instances (project "sd-board" (path "/766c70bd-1acb-59f5-b703-96c0315a8041" (reference "H1") (unit 1)))))
-(symbol (lib_id "Mechanical:MountingHole") (at 231.14 149.86 0) (unit 1) (exclude_from_sim no) (in_bom no) (on_board yes) (dnp no) (property "Reference" "H2" (at 231.14 135.86 0) (effects (font (size 1.27 1.27)))) (property "Value" "M2.5" (at 231.14 163.86 0) (effects (font (size 1.27 1.27)))) (property "Footprint" "MountingHole:MountingHole_2.7mm_M2.5" (at 231.14 149.86 0) (effects (font (size 1.27 1.27)) (hide yes))) (property "Datasheet" "" (at 231.14 149.86 0) (effects (font (size 1.27 1.27)) (hide yes))) (property "LCSC" "" (at 231.14 149.86 0) (effects (font (size 1.27 1.27)) (hide yes)))  (instances (project "sd-board" (path "/766c70bd-1acb-59f5-b703-96c0315a8041" (reference "H2") (unit 1)))))
+(symbol (lib_id "Mechanical:MountingHole") (at 215.9 149.86 0) (unit 1) (exclude_from_sim no) (in_bom no) (on_board yes) (dnp no) (property "Reference" "H1" (at 215.9 135.86 0) (effects (font (size 1.27 1.27)))) (property "Value" "pole" (at 215.9 163.86 0) (effects (font (size 1.27 1.27)))) (property "Footprint" "sdboard:PoleHole" (at 215.9 149.86 0) (effects (font (size 1.27 1.27)) (hide yes))) (property "Datasheet" "" (at 215.9 149.86 0) (effects (font (size 1.27 1.27)) (hide yes))) (property "LCSC" "" (at 215.9 149.86 0) (effects (font (size 1.27 1.27)) (hide yes)))  (instances (project "sd-board" (path "/766c70bd-1acb-59f5-b703-96c0315a8041" (reference "H1") (unit 1)))))
+(symbol (lib_id "Mechanical:MountingHole") (at 231.14 149.86 0) (unit 1) (exclude_from_sim no) (in_bom no) (on_board yes) (dnp no) (property "Reference" "H2" (at 231.14 135.86 0) (effects (font (size 1.27 1.27)))) (property "Value" "pole" (at 231.14 163.86 0) (effects (font (size 1.27 1.27)))) (property "Footprint" "sdboard:PoleHole" (at 231.14 149.86 0) (effects (font (size 1.27 1.27)) (hide yes))) (property "Datasheet" "" (at 231.14 149.86 0) (effects (font (size 1.27 1.27)) (hide yes))) (property "LCSC" "" (at 231.14 149.86 0) (effects (font (size 1.27 1.27)) (hide yes)))  (instances (project "sd-board" (path "/766c70bd-1acb-59f5-b703-96c0315a8041" (reference "H2") (unit 1)))))
 (symbol (lib_id "power:PWR_FLAG") (at 40.64 149.86 0) (unit 1) (exclude_from_sim no) (in_bom no) (on_board no) (dnp no) (property "Reference" "#FLG01" (at 40.64 135.86 0) (effects (font (size 1.27 1.27)) (hide yes))) (property "Value" "PWR_FLAG" (at 40.64 163.86 0) (effects (font (size 1.27 1.27)) (hide yes))) (property "Footprint" "" (at 40.64 149.86 0) (effects (font (size 1.27 1.27)) (hide yes))) (property "Datasheet" "" (at 40.64 149.86 0) (effects (font (size 1.27 1.27)) (hide yes))) (property "LCSC" "" (at 40.64 149.86 0) (effects (font (size 1.27 1.27)) (hide yes))) (pin "1") (instances (project "sd-board" (path "/766c70bd-1acb-59f5-b703-96c0315a8041" (reference "#FLG01") (unit 1)))))
 (label "3V3" (at 40.64 149.86 0) (effects (font (size 1.27 1.27)) (justify left bottom)))

Commit message: feat(hardware): SD board v3 on the user's caliper measurements (MEASUREMENTS.md, a to j): the poles are 6.9 mm with their centres 3.4 mm in, so they stand over the edge: two U-notches open to the left (0.6 mm play), 45.55 mm apart (the board's 46.1 and the cover's 45 differ by 1.1); 38.1 was between the poles' facing edges; the strip's top at the FM-1 board's top edge, lanes clear of the notches; no holes left
Parts:
- removed H1, H2: pole, sdboard:PoleHole, symbol Mechanical:MountingHole
Changed lines of the file:
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@@
 (label "LCD_CS" (at 226.06 96.52 180) (effects (font (size 1.27 1.27)) (justify right bottom)))
 (label "GND" (at 231.14 101.6 270) (effects (font (size 1.27 1.27)) (justify left bottom)))
-(symbol (lib_id "Mechanical:MountingHole") (at 215.9 149.86 0) (unit 1) (exclude_from_sim no) (in_bom no) (on_board yes) (dnp no) (property "Reference" "H1" (at 215.9 135.86 0) (effects (font (size 1.27 1.27)))) (property "Value" "pole" (at 215.9 163.86 0) (effects (font (size 1.27 1.27)))) (property "Footprint" "sdboard:PoleHole" (at 215.9 149.86 0) (effects (font (size 1.27 1.27)) (hide yes))) (property "Datasheet" "" (at 215.9 149.86 0) (effects (font (size 1.27 1.27)) (hide yes))) (property "LCSC" "" (at 215.9 149.86 0) (effects (font (size 1.27 1.27)) (hide yes)))  (instances (project "sd-board" (path "/766c70bd-1acb-59f5-b703-96c0315a8041" (reference "H1") (unit 1)))))
-(symbol (lib_id "Mechanical:MountingHole") (at 231.14 149.86 0) (unit 1) (exclude_from_sim no) (in_bom no) (on_board yes) (dnp no) (property "Reference" "H2" (at 231.14 135.86 0) (effects (font (size 1.27 1.27)))) (property "Value" "pole" (at 231.14 163.86 0) (effects (font (size 1.27 1.27)))) (property "Footprint" "sdboard:PoleHole" (at 231.14 149.86 0) (effects (font (size 1.27 1.27)) (hide yes))) (property "Datasheet" "" (at 231.14 149.86 0) (effects (font (size 1.27 1.27)) (hide yes))) (property "LCSC" "" (at 231.14 149.86 0) (effects (font (size 1.27 1.27)) (hide yes)))  (instances (project "sd-board" (path "/766c70bd-1acb-59f5-b703-96c0315a8041" (reference "H2") (unit 1)))))
 (symbol (lib_id "power:PWR_FLAG") (at 40.64 149.86 0) (unit 1) (exclude_from_sim no) (in_bom no) (on_board no) (dnp no) (property "Reference" "#FLG01" (at 40.64 135.86 0) (effects (font (size 1.27 1.27)) (hide yes))) (property "Value" "PWR_FLAG" (at 40.64 163.86 0) (effects (font (size 1.27 1.27)) (hide yes))) (property "Footprint" "" (at 40.64 149.86 0) (effects (font (size 1.27 1.27)) (hide yes))) (property "Datasheet" "" (at 40.64 149.86 0) (effects (font (size 1.27 1.27)) (hide yes))) (property "LCSC" "" (at 40.64 149.86 0) (effects (font (size 1.27 1.27)) (hide yes))) (pin "1") (instances (project "sd-board" (path "/766c70bd-1acb-59f5-b703-96c0315a8041" (reference "#FLG01") (unit 1)))))
 (label "3V3" (at 40.64 149.86 0) (effects (font (size 1.27 1.27)) (justify left bottom)))
