File: hardware/sd-board/sd-board.kicad_sch (KiCad schematic)
At the start: 27 parts, among them J1 TF-01A push-push, J2 FPC 10P 0.5mm (IN), J3 FPC 10P 0.5mm top contact (LC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, U1 74LVC1G04, U2 USBLC6-2SC6, U3 USBLC6-2SC6

Commit message: feat(sd-board): J2 single-sided bottom contact (XUNPU FPC-05F-10PH20, C2856798, the user's ruling), turned and wired by place as J3 (J2_AT): the mirror check settled from MEASUREMENTS.md (J12's cable gold faces the FM-1 board, round the edge it faces our board: gold DOWN at J2, J12 pin 1 on J2's first contact from the left, type A); J2 at 91.3/58.5, its ground pins to its tabs; DRC 0, nets 82 = 82, mockups regenerated (0 open edges); READMEs: a prototype ready to order, the bench tests open
Parts:
- J2: value FPC 10P 0.5mm (IN) -> FPC 10P 0.5mm bottom contact (IN); footprint sdboard:FPC-SMD_10P-P0.50_HC-FPC-05-09-10RLTAG -> sdboard:FPC-SMD_10P-P0.50_XUNPU_FPC-05F-10PH20; LCSC C5213750 -> C2856798
Connections:
- net 3V3: now also J2.4 (Pin_4); no longer J2.7 (Pin_7)
- net CLK: now also J2.7 (Pin_7); no longer J2.4 (Pin_4)
- net LCD_6: now also J2.5 (Pin_5); no longer J2.6 (Pin_6)
- net LCD_8: now also J2.3 (Pin_3); no longer J2.8 (Pin_8)
- net LCD_9: now also J2.2 (Pin_2); no longer J2.9 (Pin_9)
- net LCD_CS: now also J2.8 (Pin_8); no longer J2.3 (Pin_3)
- net MISO: now also J2.9 (Pin_9); no longer J2.2 (Pin_2)
- net MOSI: now also J2.6 (Pin_6); no longer J2.5 (Pin_5)
Changed lines of the file:
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@@
 (symbol (lib_id "Connector:TestPoint") (at 231.14 175.26 0) (unit 1) (exclude_from_sim no) (in_bom no) (on_board yes) (dnp no) (property "Reference" "TP5" (at 231.14 161.26 0) (effects (font (size 1.27 1.27)))) (property "Value" "J12 DET" (at 231.14 189.26 0) (effects (font (size 1.27 1.27)))) (property "Footprint" "TestPoint:TestPoint_Pad_D1.5mm" (at 231.14 175.26 0) (effects (font (size 1.27 1.27)) (hide yes))) (property "Datasheet" "" (at 231.14 175.26 0) (effects (font (size 1.27 1.27)) (hide yes))) (property "LCSC" "" (at 231.14 175.26 0) (effects (font (size 1.27 1.27)) (hide yes))) (pin "1") (instances (project "sd-board" (path "/766c70bd-1acb-59f5-b703-96c0315a8041" (reference "TP5") (unit 1)))))
 (label "CARD_DET" (at 231.14 175.26 270) (effects (font (size 1.27 1.27)) (justify left bottom)))
-(symbol (lib_id "Connector_Generic_MountingPin:Conn_01x10_MountingPin") (at 231.14 88.9 0) (unit 1) (exclude_from_sim no) (in_bom yes) (on_board yes) (dnp no) (property "Reference" "J2" (at 231.14 74.9 0) (effects (font (size 1.27 1.27)))) (property "Value" "FPC 10P 0.5mm (IN)" (at 231.14 102.9 0) (effects (font (size 1.27 1.27)))) (property "Footprint" "sdboard:FPC-SMD_10P-P0.50_HC-FPC-05-09-10RLTAG" (at 231.14 88.9 0) (effects (font (size 1.27 1.27)) (hide yes))) (property "Datasheet" "" (at 231.14 88.9 0) (effects (font (size 1.27 1.27)) (hide yes))) (property "LCSC" "C5213750" (at 231.14 88.9 0) (effects (font (size 1.27 1.27)) (hide yes))) (pin "1") (pin "2") (pin "3") (pin "4") (pin "5") (pin "6") (pin "7") (pin "8") (pin "9") (pin "10") (pin "MP") (instances (project "sd-board" (path "/766c70bd-1acb-59f5-b703-96c0315a8041" (reference "J2") (unit 1)))))
+(symbol (lib_id "Connector_Generic_MountingPin:Conn_01x10_MountingPin") (at 231.14 88.9 0) (unit 1) (exclude_from_sim no) (in_bom yes) (on_board yes) (dnp no) (property "Reference" "J2" (at 231.14 74.9 0) (effects (font (size 1.27 1.27)))) (property "Value" "FPC 10P 0.5mm bottom contact (IN)" (at 231.14 102.9 0) (effects (font (size 1.27 1.27)))) (property "Footprint" "sdboard:FPC-SMD_10P-P0.50_XUNPU_FPC-05F-10PH20" (at 231.14 88.9 0) (effects (font (size 1.27 1.27)) (hide yes))) (property "Datasheet" "" (at 231.14 88.9 0) (effects (font (size 1.27 1.27)) (hide yes))) (property "LCSC" "C2856798" (at 231.14 88.9 0) (effects (font (size 1.27 1.27)) (hide yes))) (pin "1") (pin "2") (pin "3") (pin "4") (pin "5") (pin "6") (pin "7") (pin "8") (pin "9") (pin "10") (pin "MP") (instances (project "sd-board" (path "/766c70bd-1acb-59f5-b703-96c0315a8041" (reference "J2") (unit 1)))))
+(label "GND" (at 226.06 101.6 180) (effects (font (size 1.27 1.27)) (justify right bottom)))
+(label "MISO" (at 226.06 99.06 180) (effects (font (size 1.27 1.27)) (justify right bottom)))
+(label "LCD_CS" (at 226.06 96.52 180) (effects (font (size 1.27 1.27)) (justify right bottom)))
+(label "CLK" (at 226.06 93.98 180) (effects (font (size 1.27 1.27)) (justify right bottom)))
+(label "MOSI" (at 226.06 91.44 180) (effects (font (size 1.27 1.27)) (justify right bottom)))
+(label "LCD_6" (at 226.06 88.9 180) (effects (font (size 1.27 1.27)) (justify right bottom)))
+(label "3V3" (at 226.06 86.36 180) (effects (font (size 1.27 1.27)) (justify right bottom)))
+(label "LCD_8" (at 226.06 83.82 180) (effects (font (size 1.27 1.27)) (justify right bottom)))
+(label "LCD_9" (at 226.06 81.28 180) (effects (font (size 1.27 1.27)) (justify right bottom)))
 (label "GND" (at 226.06 78.74 180) (effects (font (size 1.27 1.27)) (justify right bottom)))
-(label "MISO" (at 226.06 81.28 180) (effects (font (size 1.27 1.27)) (justify right bottom)))
-(label "LCD_CS" (at 226.06 83.82 180) (effects (font (size 1.27 1.27)) (justify right bottom)))
-(label "CLK" (at 226.06 86.36 180) (effects (font (size 1.27 1.27)) (justify right bottom)))
-(label "MOSI" (at 226.06 88.9 180) (effects (font (size 1.27 1.27)) (justify right bottom)))
-(label "LCD_6" (at 226.06 91.44 180) (effects (font (size 1.27 1.27)) (justify right bottom)))
-(label "3V3" (at 226.06 93.98 180) (effects (font (size 1.27 1.27)) (justify right bottom)))
-(label "LCD_8" (at 226.06 96.52 180) (effects (font (size 1.27 1.27)) (justify right bottom)))
-(label "LCD_9" (at 226.06 99.06 180) (effects (font (size 1.27 1.27)) (justify right bottom)))
-(label "GND" (at 226.06 101.6 180) (effects (font (size 1.27 1.27)) (justify right bottom)))
 (label "GND" (at 231.14 106.68 270) (effects (font (size 1.27 1.27)) (justify left bottom)))
 (symbol (lib_id "Connector_Generic_MountingPin:Conn_01x10_MountingPin") (at 259.08 88.9 0) (unit 1) (exclude_from_sim no) (in_bom yes) (on_board yes) (dnp no) (property "Reference" "J3" (at 259.08 74.9 0) (effects (font (size 1.27 1.27)))) (property "Value" "FPC 10P 0.5mm top contact (LCD)" (at 259.08 102.9 0) (effects (font (size 1.27 1.27)))) (property "Footprint" "sdboard:FPC-SMD_10P-P0.50_XUNPU_FPC-0.5AS-10PWBH20" (at 259.08 88.9 0) (effects (font (size 1.27 1.27)) (hide yes))) (property "Datasheet" "" (at 259.08 88.9 0) (effects (font (size 1.27 1.27)) (hide yes))) (property "LCSC" "C3446068" (at 259.08 88.9 0) (effects (font (size 1.27 1.27)) (hide yes))) (pin "1") (pin "2") (pin "3") (pin "4") (pin "5") (pin "6") (pin "7") (pin "8") (pin "9") (pin "10") (pin "MP") (instances (project "sd-board" (path "/766c70bd-1acb-59f5-b703-96c0315a8041" (reference "J3") (unit 1)))))
